File: schematics/usb-dac/dac_mcu_usb.sch (KiCad schematic (older format))
At the start: 2 parts

Commit message: Added clock, missing buffered output
Parts:
- R? (x2): symbol Device:R -> usb-dac-rescue:R-Device
Changed lines of the file:
@@
 EESchema Schematic File Version 4
+LIBS:usb-dac-cache
 EELAYER 26 0
 EELAYER END
@@
 $EndDescr
 $Comp
-L Device:R R?
+L usb-dac-rescue:R-Device R?
 U 1 1 5B2D8668
 P 3650 2150
@@
 $EndComp
 $Comp
-L Device:R R?
+L usb-dac-rescue:R-Device R?
 U 1 1 5B2D86AD
 P 3650 2300
