File: schematics/usb-dac/dac_mcu_usb.sch (KiCad schematic (older format))
At the start: 2 parts

Commit message: Preparing Merging
Parts:
- removed R? (x2): R, symbol Device:R
- added C? (x2): C_Small, Capacitors_SMD:C_0603, symbol Device:C_Small
- added ESD? (x2): PGB1010603MR, Package_TO_SOT_SMD:SOT-23, symbol my_dac:PGB1010603MR
- added J?: AVR-JTAG-10, symbol Connector:AVR-JTAG-10
- added J?: USB_B, symbol Connector:USB_B
- added L?: Ferrite_Bead_Small, symbol Device:Ferrite_Bead_Small
- added R? (x3): R, Resistors_SMD:R_0603, symbol Device:R
- added U? (x5): AT32UC3A3256, symbol my_dac:AT32UC3A3256
Connections:
- net labels added: GND, VBUS, VDD_+3V3
- wire segments 0 -> 49
