File: schematics/usb-dac/dac_clocks.sch (KiCad schematic (older format))
At the start: 0 parts

Commit message: Added clock, missing buffered output
Parts:
- added R? (x10): R, Resistors_SMD:R_0603, symbol device:R
- added R? (x3): R, symbol device:R
- added U?: 74LVC1G00, symbol my_dac:74LVC1G00
- added X? (x2): GXO-7531-B, Oscillators:Oscillator_SMD_Golledge-GXO7531-4pin_7.0x5.0mm, symbol my_dac:GXO-7531-B
Connections:
- net labels added: GND, MCLK_MCU, MCLK_P48_N441, PCM5102_MCLK, VDD_X02
- wire segments 0 -> 34

Commit message: Merged and fix merge errors
Parts:
- R? (x13): symbol device:R -> usb-dac-rescue:R-device
Changed lines of the file:
@@
 $EndComp
 $Comp
-L device:R R?
+L usb-dac-rescue:R-device R?
 U 1 1 5B31977F
 P 3950 1400
@@
 $EndComp
 $Comp
-L device:R R?
+L usb-dac-rescue:R-device R?
 U 1 1 5B3197CE
 P 3950 1600
@@
 $EndComp
 $Comp
-L device:R R?
+L usb-dac-rescue:R-device R?
 U 1 1 5B319BFE
 P 3950 2800
@@
 $EndComp
 $Comp
-L device:R R?
+L usb-dac-rescue:R-device R?
 U 1 1 5B319C04
 P 3950 3000
@@
 MCLK_P48_N441
 $Comp
-L device:R R?
+L usb-dac-rescue:R-device R?
 U 1 1 5B31A20E
 P 2100 950
@@
 $EndComp
 $Comp
-L device:R R?
+L usb-dac-rescue:R-device R?
 U 1 1 5B31B616
 P 5450 1400
@@
 $EndComp
 $Comp
-L device:R R?
+L usb-dac-rescue:R-device R?
 U 1 1 5B31B64F
 P 5450 2800
@@
 PCM5102_MCLK
 $Comp
-L device:R R?
+L usb-dac-rescue:R-device R?
 U 1 1 5B31B795
 P 6200 1400
@@
 $EndComp
 $Comp
-L device:R R?
+L usb-dac-rescue:R-device R?
 U 1 1 5B31B7CB
 P 6750 1400
@@
 $EndComp
 $Comp
-L device:R R?
+L usb-dac-rescue:R-device R?
 U 1 1 5B31B800
 P 7950 1700
@@
 MCLK_MCU
 $Comp
-L device:R R?
+L usb-dac-rescue:R-device R?
 U 1 1 5B31DFAA
 P 10350 1400
@@
 $EndComp
 $Comp
-L device:R R?
+L usb-dac-rescue:R-device R?
 U 1 1 5B31DFFD
 P 10350 1900
@@
 $EndComp
 $Comp
-L device:R R?
+L usb-dac-rescue:R-device R?
 U 1 1 5B31E033
 P 10350 2100
