File: schematics/usb-dac/dac_in_out.sch (KiCad schematic (older format))
At the start: 31 parts

Commit message: Added clock, missing buffered output
Parts:
- C? (x14): symbol Device:C_Small -> usb-dac-rescue:C_Small-Device
- C? (x4): symbol Device:CP1_Small -> usb-dac-rescue:CP1_Small-Device
- D?: symbol Device:LED_Dual_ACA -> usb-dac-rescue:LED_Dual_ACA-Device
- J?: symbol Connector:Conn_Coaxial_x2 -> usb-dac-rescue:Conn_Coaxial_x2-Connector
- R? (x9): symbol Device:R -> usb-dac-rescue:R-Device
- U?: symbol Analog_DAC:AK4430ET -> usb-dac-rescue:AK4430ET-Analog_DAC
Changed lines of the file:
@@
 EESchema Schematic File Version 4
+LIBS:usb-dac-cache
 EELAYER 26 0
 EELAYER END
@@
 $EndDescr
 $Comp
-L Device:LED_Dual_ACA D?
+L usb-dac-rescue:LED_Dual_ACA-Device D?
 U 1 1 5B28ABFB
 P 1500 1150
@@
 $EndComp
 $Comp
-L Device:R R?
+L usb-dac-rescue:R-Device R?
 U 1 1 5B28AC73
 P 2100 1050
@@
 $EndComp
 $Comp
-L Device:R R?
+L usb-dac-rescue:R-Device R?
 U 1 1 5B28ACAC
 P 2100 1250
@@
 $EndComp
 $Comp
-L Device:R R?
+L usb-dac-rescue:R-Device R?
 U 1 1 5B28AECC
 P 2550 1250
@@
 	2800 1050 2250 1050
 $Comp
-L Analog_DAC:AK4430ET U?
+L usb-dac-rescue:AK4430ET-Analog_DAC U?
 U 1 1 5B28B76D
 P 4400 4650
@@
 $EndComp
 $Comp
-L Device:R R?
+L usb-dac-rescue:R-Device R?
 U 1 1 5B28B8A3
 P 3350 5000
@@
 $EndComp
 $Comp
-L Device:R R?
+L usb-dac-rescue:R-Device R?
 U 1 1 5B28B946
 P 3350 4850
@@
 $EndComp
 $Comp
-L Device:R R?
+L usb-dac-rescue:R-Device R?
 U 1 1 5B28B968
 P 3350 4700
@@
 $EndComp
 $Comp
-L Device:R R?
+L usb-dac-rescue:R-Device R?
 U 1 1 5B28B990
 P 3350 4550
@@
 	3200 4550 3000 4550
 $Comp
-L Device:C_Small C?
+L usb-dac-rescue:C_Small-Device C?
 U 1 1 5B28CDC6
 P 3300 4100
@@
 $EndComp
 $Comp
-L Device:C_Small C?
+L usb-dac-rescue:C_Small-Device C?
 U 1 1 5B28CDF9
 P 2850 4100
@@
 $EndComp
 $Comp
-L Device:C_Small C?
+L usb-dac-rescue:C_Small-Device C?
 U 1 1 5B28DFE0
 P 5500 5450
@@
 $EndComp
 $Comp
-L Device:CP1_Small C?
+L usb-dac-rescue:CP1_Small-Device C?
 U 1 1 5B28E09B
 P 5950 5450
@@
 	3300 3900 2850 3900
 $Comp
-L Device:R R?
+L usb-dac-rescue:R-Device R?
 U 1 1 5B291F72
 P 6300 5150
@@
 $EndComp
 $Comp
-L Device:R R?
+L usb-dac-rescue:R-Device R?
 U 1 1 5B292023
 P 6300 5000
@@
 	6150 5150 5000 5150
 $Comp
-L Connector:Conn_Coaxial_x2 J?
+L usb-dac-rescue:Conn_Coaxial_x2-Connector J?
 U 1 1 5B293415
 P 8500 4550
@@
 $EndComp
 $Comp
-L Device:C_Small C?
+L usb-dac-rescue:C_Small-Device C?
 U 1 1 5B29353A
 P 7100 5450
@@
 $EndComp
 $Comp
-L Device:C_Small C?
+L usb-dac-rescue:C_Small-Device C?
 U 1 1 5B2936CE
 P 7500 5450
@@
 	8900 4550 8800 4550
 $Comp
-L Device:C_Small C?
+L usb-dac-rescue:C_Small-Device C?
 U 1 1 5B298857
 P 6350 2350
@@
 $EndComp
 $Comp
-L Device:C_Small C?
+L usb-dac-rescue:C_Small-Device C?
 U 1 1 5B29897E
 P 6350 3300
@@
 $EndComp
 $Comp
-L Device:C_Small C?
+L usb-dac-rescue:C_Small-Device C?
 U 1 1 5B2989C8
 P 6350 4250
@@
 $EndComp
 $Comp
-L Device:C_Small C?
+L usb-dac-rescue:C_Small-Device C?
 U 1 1 5B298A22
 P 6900 2350
@@
 $EndComp
 $Comp
-L Device:C_Small C?
+L usb-dac-rescue:C_Small-Device C?
 U 1 1 5B298AC8
 P 6900 3300
@@
 $EndComp
 $Comp
-L Device:C_Small C?
+L usb-dac-rescue:C_Small-Device C?
 U 1 1 5B298B14
 P 6900 4250
@@
 $EndComp
 $Comp
-L Device:C_Small C?
+L usb-dac-rescue:C_Small-Device C?
 U 1 1 5B298B7E
 P 7400 2350
@@
 $EndComp
 $Comp
-L Device:C_Small C?
+L usb-dac-rescue:C_Small-Device C?
 U 1 1 5B298C51
 P 7400 3300
@@
 $EndComp
 $Comp
-L Device:C_Small C?
+L usb-dac-rescue:C_Small-Device C?
 U 1 1 5B298CA3
 P 7400 4250
@@
 $EndComp
 $Comp
-L Device:CP1_Small C?
+L usb-dac-rescue:CP1_Small-Device C?
 U 1 1 5B298D0C
 P 7850 2350
@@
 $EndComp
 $Comp
-L Device:CP1_Small C?
+L usb-dac-rescue:CP1_Small-Device C?
 U 1 1 5B298E00
 P 7850 3300
@@
 $EndComp
 $Comp
-L Device:CP1_Small C?
+L usb-dac-rescue:CP1_Small-Device C?
 U 1 1 5B298E64
 P 7850 4250
